Commit message: Changed camera position in URDF to face the ground.
Added a depth camera sensor plugin to get posistion of the mine relative to the odom frame.
Posistion of the mine can be obtained using tf and in the camera frame by using
rosrun find_object_2d print_objects_detected node.

The chetak_wc_Camera description urdf mass,torque and inertia values have been reduced by a factor of 10.
Base link had a mass of 600kg before reduction, need to hollow out the bot in cad and change material properties.

Modified minefield.launch in mine_field package to launch all necessary nodes.

Adding markers in 2d costmap at detected coordinates and integration into nav stack yet to be done.

File: src/chetak_wc_Wheel_bug_description/urdf/chetak_wc_Wheel_bug.xacro (robot description, xacro)
@@ -1,17 +1,17 @@
 <?xml version="1.0" ?>
-<robot name="chetak_wc_Camera" xmlns:xacro="http://www.ros.org/wiki/xacro">
-<xacro:include filename="$(find chetak_wc_Camera_description)/urdf/materials.xacro" />
-<xacro:include filename="$(find chetak_wc_Camera_description)/urdf/chetak_wc_Camera.trans" />
-<xacro:include filename="$(find chetak_wc_Camera_description)/urdf/chetak_wc_Camera.gazebo" />
+<robot name="chetak_wc_Wheel_bug" xmlns:xacro="http://www.ros.org/wiki/xacro">
+<xacro:include filename="$(find chetak_wc_Wheel_bug_description)/urdf/materials.xacro" />
+<xacro:include filename="$(find chetak_wc_Wheel_bug_description)/urdf/chetak_wc_Wheel_bug.trans" />
+<xacro:include filename="$(find chetak_wc_Wheel_bug_description)/urdf/chetak_wc_Wheel_bug.gazebo" />
 <link name="base_link">
   <inertial>
     <origin rpy="0 0 0" xyz="-0.36835618355447514 0.19999999999999993 0.20351102142822705"/>
-    <mass value="67.27916543636255"/>
-    <inertia ixx="1.6448418" ixy="0.0" ixz="0.0686477" iyy="2.773513" iyz="0.0" izz="2.9814385"/>
+    <mass value="672.7916543636255"/>
+    <inertia ixx="16.448418" ixy="0.0" ixz="0.686477" iyy="27.73513" iyz="-0.0" izz="29.814385"/>
   </inertial>
   <visual>
     <origin rpy="0 0 0" xyz="0 0 0"/>
     <geometry>
-      <mesh filename="package://chetak_wc_Camera_description/meshes/base_link.stl" scale="0.001 0.001 0.001"/>
+      <mesh filename="package://chetak_wc_Wheel_bug_description/meshes/base_link.stl" scale="0.001 0.001 0.001"/>
     </geometry>
     <material name="silver"/>
@@ -20,5 +20,5 @@
     <origin rpy="0 0 0" xyz="0 0 0"/>
     <geometry>
-      <mesh filename="package://chetak_wc_Camera_description/meshes/base_link.stl" scale="0.001 0.001 0.001"/>
+      <mesh filename="package://chetak_wc_Wheel_bug_description/meshes/base_link.stl" scale="0.001 0.001 0.001"/>
     </geometry>
   </collision>
@@ -33,5 +33,5 @@
     <origin rpy="0 0 0" xyz="0.525 0.08 -0.075"/>
     <geometry>
-      <mesh filename="package://chetak_wc_Camera_description/meshes/b_r_1.stl" scale="0.001 0.001 0.001"/>
+      <mesh filename="package://chetak_wc_Wheel_bug_description/meshes/b_r_1.stl" scale="0.001 0.001 0.001"/>
     </geometry>
     <material name="silver"/>
@@ -40,5 +40,5 @@
     <origin rpy="0 0 0" xyz="0.525 0.08 -0.075"/>
     <geometry>
-      <mesh filename="package://chetak_wc_Camera_description/meshes/b_r_1.stl" scale="0.001 0.001 0.001"/>
+      <mesh filename="package://chetak_wc_Wheel_bug_description/meshes/b_r_1.stl" scale="0.001 0.001 0.001"/>
     </geometry>
   </collision>
@@ -53,5 +53,5 @@
     <origin rpy="0 0 0" xyz="0.175 -0.48 -0.075"/>
     <geometry>
-      <mesh filename="package://chetak_wc_Camera_description/meshes/f_l_1.stl" scale="0.001 0.001 0.001"/>
+      <mesh filename="package://chetak_wc_Wheel_bug_description/meshes/f_l_1.stl" scale="0.001 0.001 0.001"/>
     </geometry>
     <material name="silver"/>
@@ -60,5 +60,5 @@
     <origin rpy="0 0 0" xyz="0.175 -0.48 -0.075"/>
     <geometry>
-      <mesh filename="package://chetak_wc_Camera_description/meshes/f_l_1.stl" scale="0.001 0.001 0.001"/>
+      <mesh filename="package://chetak_wc_Wheel_bug_description/meshes/f_l_1.stl" scale="0.001 0.001 0.001"/>
     </geometry>
   </collision>
@@ -73,5 +73,5 @@
     <origin rpy="0 0 0" xyz="0.175 0.08 -0.075"/>
     <geometry>
-      <mesh filename="package://chetak_wc_Camera_description/meshes/f_r_1.stl" scale="0.001 0.001 0.001"/>
+      <mesh filename="package://chetak_wc_Wheel_bug_description/meshes/f_r_1.stl" scale="0.001 0.001 0.001"/>
     </geometry>
     <material name="silver"/>
@@ -80,5 +80,5 @@
     <origin rpy="0 0 0" xyz="0.175 0.08 -0.075"/>
     <geometry>
-      <mesh filename="package://chetak_wc_Camera_description/meshes/f_r_1.stl" scale="0.001 0.001 0.001"/>
+      <mesh filename="package://chetak_wc_Wheel_bug_description/meshes/f_r_1.stl" scale="0.001 0.001 0.001"/>
     </geometry>
   </collision>
@@ -93,5 +93,5 @@
     <origin rpy="0 0 0" xyz="0.525 -0.48 -0.075"/>
     <geometry>
-      <mesh filename="package://chetak_wc_Camera_description/meshes/b_l_1.stl" scale="0.001 0.001 0.001"/>
+      <mesh filename="package://chetak_wc_Wheel_bug_description/meshes/b_l_1.stl" scale="0.001 0.001 0.001"/>
     </geometry>
     <material name="silver"/>
@@ -100,5 +100,5 @@
     <origin rpy="0 0 0" xyz="0.525 -0.48 -0.075"/>
     <geometry>
-      <mesh filename="package://chetak_wc_Camera_description/meshes/b_l_1.stl" scale="0.001 0.001 0.001"/>
+      <mesh filename="package://chetak_wc_Wheel_bug_description/meshes/b_l_1.stl" scale="0.001 0.001 0.001"/>
     </geometry>
   </collision>
@@ -113,12 +113,12 @@
     <origin rpy="0 0 0" xyz="0.40087 -0.2 -0.32"/>
     <geometry>
-      <mesh filename="package://chetak_wc_Camera_description/meshes/uvc_rod__1.stl" scale="0.001 0.001 0.001"/>
-    </geometry>
-    <material name="silver"/>
-  </visual>
-  <collision>
-    <origin rpy="0 0 0" xyz="0.40087 -0.2 -0.32"/>
-    <geometry>
-      <mesh filename="package://chetak_wc_Camera_description/meshes/uvc_rod__1.stl" scale="0.001 0.001 0.001"/>
+      <mesh filename="package://chetak_wc_Wheel_bug_description/meshes/uvc_rod__1.stl" scale="0.001 0.001 0.001"/>
+    </geometry>
+    <material name="silver"/>
+  </visual>
+  <collision>
+    <origin rpy="0 0 0" xyz="0.40087 -0.2 -0.32"/>
+    <geometry>
+      <mesh filename="package://chetak_wc_Wheel_bug_description/meshes/uvc_rod__1.stl" scale="0.001 0.001 0.001"/>
     </geometry>
   </collision>
@@ -133,12 +133,12 @@
     <origin rpy="0 0 0" xyz="0.40087 -0.2 -0.32"/>
     <geometry>
-      <mesh filename="package://chetak_wc_Camera_description/meshes/uvc_plate_1.stl" scale="0.001 0.001 0.001"/>
-    </geometry>
-    <material name="silver"/>
-  </visual>
-  <collision>
-    <origin rpy="0 0 0" xyz="0.40087 -0.2 -0.32"/>
-    <geometry>
-      <mesh filename="package://chetak_wc_Camera_description/meshes/uvc_plate_1.stl" scale="0.001 0.001 0.001"/>
+      <mesh filename="package://chetak_wc_Wheel_bug_description/meshes/uvc_plate_1.stl" scale="0.001 0.001 0.001"/>
+    </geometry>
+    <material name="silver"/>
+  </visual>
+  <collision>
+    <origin rpy="0 0 0" xyz="0.40087 -0.2 -0.32"/>
+    <geometry>
+      <mesh filename="package://chetak_wc_Wheel_bug_description/meshes/uvc_plate_1.stl" scale="0.001 0.001 0.001"/>
     </geometry>
   </collision>
@@ -153,5 +153,5 @@
     <origin rpy="0 0 0" xyz="0.015464 -0.2 -0.156443"/>
     <geometry>
-      <mesh filename="package://chetak_wc_Camera_description/meshes/lidar_1.stl" scale="0.001 0.001 0.001"/>
+      <mesh filename="package://chetak_wc_Wheel_bug_description/meshes/lidar_1.stl" scale="0.001 0.001 0.001"/>
     </geometry>
     <material name="silver"/>
@@ -160,5 +160,25 @@
     <origin rpy="0 0 0" xyz="0.015464 -0.2 -0.156443"/>
     <geometry>
-      <mesh filename="package://chetak_wc_Camera_description/meshes/lidar_1.stl" scale="0.001 0.001 0.001"/>
+      <mesh filename="package://chetak_wc_Wheel_bug_description/meshes/lidar_1.stl" scale="0.001 0.001 0.001"/>
+    </geometry>
+  </collision>
+</link>
+<link name="camera_1">
+  <inertial>
+    <origin rpy="0 0 0" xyz="-0.02247030893236321 -1.4652168367490503e-13 0.023484452064101102"/>
+    <mass value="2.814971712983161"/>
+    <inertia ixx="0.005636" ixy="0.0" ixz="-8e-05" iyy="0.001135" iyz="0.0" izz="0.005704"/>
+  </inertial>
+  <visual>
+    <origin rpy="0 0 0" xyz="0.175 -0.2 -0.4"/>
+    <geometry>
+      <mesh filename="package://chetak_wc_Wheel_bug_description/meshes/camera_1.stl" scale="0.001 0.001 0.001"/>
+    </geometry>
+    <material name="silver"/>
+  </visual>
+  <collision>
+    <origin rpy="0 0 0" xyz="0.175 -0.2 -0.4"/>
+    <geometry>
+      <mesh filename="package://chetak_wc_Wheel_bug_description/meshes/camera_1.stl" scale="0.001 0.001 0.001"/>
     </geometry>
   </collision>
@@ -173,5 +193,5 @@
     <origin rpy="0 0 0" xyz="0.094915 -0.2 -0.297034"/>
     <geometry>
-      <mesh filename="package://chetak_wc_Camera_description/meshes/name_1.stl" scale="0.001 0.001 0.001"/>
+      <mesh filename="package://chetak_wc_Wheel_bug_description/meshes/name_1.stl" scale="0.001 0.001 0.001"/>
     </geometry>
     <material name="silver"/>
@@ -180,25 +200,5 @@
     <origin rpy="0 0 0" xyz="0.094915 -0.2 -0.297034"/>
     <geometry>
-      <mesh filename="package://chetak_wc_Camera_description/meshes/name_1.stl" scale="0.001 0.001 0.001"/>
-    </geometry>
-  </collision>
-</link>
-<link name="camera_1">
-  <inertial>
-    <origin rpy="0 1.5708 0" xyz="-0.016515433336358125 -1.4652168367490503e-13 -0.027529353548188"/>
-    <mass value="2.814971712983161"/>
-    <inertia ixx="0.005704" ixy="0.0" ixz="8e-05" iyy="0.001135" iyz="-0.0" izz="0.005636"/>
-  </inertial>
-  <visual>
-    <origin rpy="0 0 0" xyz="-0.034536 -0.2 -0.154443"/>
-    <geometry>
-      <mesh filename="package://chetak_wc_Camera_description/meshes/camera_1.stl" scale="0.001 0.001 0.001"/>
-    </geometry>
-    <material name="silver"/>
-  </visual>
-  <collision>
-    <origin rpy="0 0 0" xyz="-0.034536 -0.2 -0.154443"/>
-    <geometry>
-      <mesh filename="package://chetak_wc_Camera_description/meshes/camera_1.stl" scale="0.001 0.001 0.001"/>
+      <mesh filename="package://chetak_wc_Wheel_bug_description/meshes/name_1.stl" scale="0.001 0.001 0.001"/>
     </geometry>
   </collision>
@@ -243,4 +243,9 @@
   <child link="lidar_1"/>
 </joint>
+<joint name="Rigid14" type="fixed">
+  <origin rpy="0 0 0" xyz="-0.175 0.2 0.4"/>
+  <parent link="base_link"/>
+  <child link="camera_1"/>
+</joint>
 <joint name="Rigid15" type="fixed">
   <origin rpy="0 0 0" xyz="-0.094915 0.2 0.297034"/>
@@ -248,8 +253,3 @@
   <child link="name_1"/>
 </joint>
-<joint name="Rigid16" type="fixed">
-  <origin rpy="0 1.5708 0" xyz="0.05 0.0 -0.002"/>
-  <parent link="lidar_1"/>
-  <child link="camera_1"/>
-</joint>
 </robot>
